File: matrix.sch (KiCad schematic (older format))
At the start: 134 parts, among them SW1 SW_Push, SW10 SW_Push, SW11 SW_Push, SW12 SW_Push, SW13 SW_Push, SW14 SW_Push, SW15 SW_Push, SW16 SW_Push, SW17 SW_Push, SW18 SW_Push, SW19 SW_Push, SW2 SW_Push, SW20 SW_Push, SW21 SW_Push, SW22 SW_Push, SW23 SW_Push, SW24 SW_Push, SW25 SW_Push, SW26 SW_Push, SW27 SW_Push, SW28 SW_Push, SW29 SW_Push, SW3 SW_Push, SW30 SW_Push, SW31 SW_Push, SW32 SW_Push, SW33 SW_Push, SW34 SW_Push, SW35 SW_Push, SW36 SW_Push, SW37 SW_Push, SW38 SW_Push, SW39 SW_Push, SW4 SW_Push, SW40 SW_Push, SW41 SW_Push, SW42 SW_Push, SW43 SW_Push, SW44 SW_Push, SW45 SW_Push, SW46 SW_Push, SW47 SW_Push, SW48 SW_Push, SW49 SW_Push, SW5 SW_Push, SW50 SW_Push, SW51 SW_Push, SW52 SW_Push, SW53 SW_Push, SW54 SW_Push, SW55 SW_Push, SW56 SW_Push, SW57 SW_Push, SW58 SW_Push, SW59 SW_Push, SW6 SW_Push, SW60 SW_Push, SW61 SW_Push, SW62 SW_Push, SW63 SW_Push, SW64 SW_Push, SW65 SW_Push, SW66 SW_Push, SW67 SW_Push, SW7 SW_Push, SW8 SW_Push, SW9 SW_Push

Commit message: finished assign component
Parts:
- D1, D10, D11, D12, D13, D14, D15, D16, D17, D18, D19, D2, D20, D21, D22, D23, D24, D25, D26, D27, D28, D29, D3, D30, D31, D32, D33, D34, D35, D36, D37, D38, D39, D4, D40, D41, D42, D43, D44, D45, D46, D47, D48, D49, D5, D50, D51, D52, D53, D54, D55, D56, D57, D58, D59, D6, D60, D61, D62, D63, D64, D65, D66, D67, D7, D8, D9: footprint (none) -> Diode_SMD:D_SOD-123
- SW1: footprint Esc -> MX_Only:MXOnly-1U-Hotswap
- SW10: footprint #9 -> MX_Only:MXOnly-1U-Hotswap
- SW11: footprint #0 -> MX_Only:MXOnly-1U-Hotswap
- SW12: footprint - -> MX_Only:MXOnly-1U-Hotswap
- SW13: footprint + -> MX_Only:MXOnly-1U-Hotswap
- SW14: footprint Bcksp -> MX_Only:MXOnly-2U-Hotswap
- SW15: footprint Del -> MX_Only:MXOnly-1U-Hotswap
- SW16: footprint Tab -> MX_Only:MXOnly-1.5U-Hotswap
- SW17: footprint q -> MX_Only:MXOnly-1U-Hotswap
- SW18: footprint w -> MX_Only:MXOnly-1U-Hotswap
- SW19: footprint e -> MX_Only:MXOnly-1U-Hotswap
- SW2: footprint #1 -> MX_Only:MXOnly-1U-Hotswap
- SW20: footprint r -> MX_Only:MXOnly-1U-Hotswap
- SW21: footprint t -> MX_Only:MXOnly-1U-Hotswap
- SW22: footprint y -> MX_Only:MXOnly-1U-Hotswap
- SW23: footprint u -> MX_Only:MXOnly-1U-Hotswap
- SW24: footprint i -> MX_Only:MXOnly-1U-Hotswap
- SW25: footprint o -> MX_Only:MXOnly-1U-Hotswap
- SW26: footprint p -> MX_Only:MXOnly-1U-Hotswap
- SW27: footprint [ -> MX_Only:MXOnly-1U-Hotswap
- SW28: footprint ] -> MX_Only:MXOnly-1U-Hotswap
- SW29: footprint \\ -> MX_Only:MXOnly-1.5U-Hotswap
- SW3: footprint #2 -> MX_Only:MXOnly-1U-Hotswap
- SW30: footprint Pg Up -> MX_Only:MXOnly-1.75U-Hotswap
- SW31: footprint Caps Lck -> MX_Only:MXOnly-1U-Hotswap
- SW32: footprint a -> MX_Only:MXOnly-1U-Hotswap
- SW33: footprint s -> MX_Only:MXOnly-1U-Hotswap
- SW34: footprint d -> MX_Only:MXOnly-1U-Hotswap
- SW35: footprint f -> MX_Only:MXOnly-1U-Hotswap
- SW36: footprint g -> MX_Only:MXOnly-1U-Hotswap
- SW37: footprint h -> MX_Only:MXOnly-1U-Hotswap
- SW38: footprint j -> MX_Only:MXOnly-1U-Hotswap
- SW39: footprint k -> MX_Only:MXOnly-1U-Hotswap
- SW4: footprint #3 -> MX_Only:MXOnly-1U-Hotswap
- SW40: footprint l -> MX_Only:MXOnly-1U-Hotswap
- SW41: footprint ; -> MX_Only:MXOnly-1U-Hotswap
- SW42: footprint ' -> MX_Only:MXOnly-1U-Hotswap
- SW43: footprint Enter -> MX_Only:MXOnly-2.25U-Hotswap
- SW44: footprint Pg Down -> MX_Only:MXOnly-1U-Hotswap
- SW45: footprint Shift -> MX_Only:MXOnly-2.25U-Hotswap
- SW46: footprint z -> MX_Only:MXOnly-1U-Hotswap
- SW47: footprint x -> MX_Only:MXOnly-1U-Hotswap
- SW48: footprint c -> MX_Only:MXOnly-1U-Hotswap
- SW49: footprint v -> MX_Only:MXOnly-1U-Hotswap
- SW5: footprint #4 -> MX_Only:MXOnly-1U-Hotswap
- SW50: footprint b -> MX_Only:MXOnly-1U-Hotswap
- SW51: footprint n -> MX_Only:MXOnly-1U-Hotswap
- SW52: footprint m -> MX_Only:MXOnly-1U-Hotswap
- SW53: footprint , -> MX_Only:MXOnly-1U-Hotswap
- SW54: footprint . -> MX_Only:MXOnly-1U-Hotswap
- SW55: footprint / -> MX_Only:MXOnly-1U-Hotswap
- SW56: footprint Shift -> MX_Only:MXOnly-1.75U-Hotswap
- SW57: footprint Up -> MX_Only:MXOnly-1U-Hotswap
- SW58: footprint Fn -> MX_Only:MXOnly-1U-Hotswap
- SW59: footprint Ctrl -> MX_Only:MXOnly-1.25U-Hotswap
- SW6: footprint #5 -> MX_Only:MXOnly-1U-Hotswap
- SW60, SW63: footprint Win -> MX_Only:MXOnly-1.25U-Hotswap
- SW61, SW64: footprint Alt -> MX_Only:MXOnly-1.25U-Hotswap
- SW62: footprint Space -> MX_Only:MXOnly-6.25U-Hotswap
- SW65: footprint Left -> MX_Only:MXOnly-1U-Hotswap
- SW66: footprint Down -> MX_Only:MXOnly-1U-Hotswap
- SW67: footprint Right -> MX_Only:MXOnly-1U-Hotswap
- SW7: footprint #6 -> MX_Only:MXOnly-1U-Hotswap
- SW8: footprint #7 -> MX_Only:MXOnly-1U-Hotswap
- SW9: footprint #8 -> MX_Only:MXOnly-1U-Hotswap
